Commit message: OAK-D-S2追加のためurdf修正

File: stepbot_description/urdf/stepbot.xacro (robot description, xacro)
@@ -13,5 +13,5 @@
    <origin xyz="0 0 0.0255" rpy="0 0 0"/>
    <geometry>
-    <box size="0.120 0.120 0.10"/>
+    <box size="0.130 0.120 0.10"/>
    </geometry>
    <material name="blue">
@@ -21,5 +21,5 @@
   <collision>
    <geometry>
-    <box size="0.120 0.120 0.10"/>
+    <box size="0.130 0.120 0.10"/>
    </geometry>
   </collision>
@@ -76,5 +76,5 @@
   <parent link="base_link"/>
   <child link="base_scan"/>
-  <origin xyz="0.03 0 0.115" rpy="0 0 0"/>
+  <origin xyz="0.03 0 0.114" rpy="0 0 0"/>
  </joint>
  <link name="base_scan">
@@ -94,3 +94,15 @@
   </collision>
  </link>
+<!-- include OAK-D S2 -->
+ <xacro:include filename="$(find depthai_descriptions)/urdf/include/depthai_macro.urdf.xacro"/>
+ <joint name="oak_joint" type="fixed">
+  <parent link="base_link"/>
+  <child link="oak-d-base-frame"/>
+  <origin xyz="0.08 0 0.095" rpy="0 0 0"/>
+ </joint>
+ <link name="oak-d-base-frame" />
+ <xacro:depthai_camera camera_name= "oak" camera_model = "OAK-D-S2"
+                       base_frame = "oak-d_frame" parent="oak-d-base-frame"
+                       cam_pos_x = "0" cam_pos_y = "0" cam_pos_z = "0"
+                       cam_roll = "0" cam_pitch = "0" cam_yaw = "0"/>
 </robot>
